Commit message: change views

File: src/pepper_description/urdf/pepper1.0_generated_urdf/pepperGazebo.xacro (robot description, xacro)
@@ -150,5 +150,4 @@
         <selfCollide>false</selfCollide>
         <turnGravityOff>false</turnGravityOff>
-	<material>Gazebo/Blue</material>
     </gazebo>
     <gazebo reference="LElbow">
@@ -187,5 +186,4 @@
         <selfCollide>false</selfCollide>
         <turnGravityOff>false</turnGravityOff>
-	<material>Gazebo/Blue</material>
     </gazebo>
     <gazebo reference="RElbow">

Commit message: change delay to queue method

File: src/pepper_description/urdf/pepper1.0_generated_urdf/pepperGazebo.xacro (robot description, xacro)
@@ -150,4 +150,5 @@
         <selfCollide>false</selfCollide>
         <turnGravityOff>false</turnGravityOff>
+	<material>Gazebo/Orange</material>
     </gazebo>
     <gazebo reference="LElbow">
@@ -186,4 +187,5 @@
         <selfCollide>false</selfCollide>
         <turnGravityOff>false</turnGravityOff>
+	<material>Gazebo/Orange</material>
     </gazebo>
     <gazebo reference="RElbow">

Commit message: adjust world, color a little bit

File: src/pepper_description/urdf/pepper1.0_generated_urdf/pepperGazebo.xacro (robot description, xacro)
@@ -150,5 +150,5 @@
         <selfCollide>false</selfCollide>
         <turnGravityOff>false</turnGravityOff>
-	<material>Gazebo/Orange</material>
+	<material>Gazebo/Green</material>
     </gazebo>
     <gazebo reference="LElbow">
@@ -187,5 +187,5 @@
         <selfCollide>false</selfCollide>
         <turnGravityOff>false</turnGravityOff>
-	<material>Gazebo/Orange</material>
+	<material>Gazebo/Green</material>
     </gazebo>
     <gazebo reference="RElbow">
